File: Schematics/ESP32_CAN_Board/Power.kicad_sch (KiCad schematic)
At the start: 5 parts, among them U7 LDL1117-3.3

Commit message: initial design completed
Connections:
- net ESPPower renamed +3.3V
