File: Schematics/ESP32_CAN_Board/ESP32_CAN_Board.kicad_sch (KiCad schematic)
At the start: 0 parts

Commit message: finished ready for order
Parts:
- added R1, R6: 27r, Resistor_SMD:R_0805_2012Metric_Pad1.20x1.40mm_HandSolder, symbol Device:R
Connections:
- net MCU/D+: now also R1.1
- net MCU/D-: now also R6.1
- new net USBC/D+: R1.2
- new net USBC/D-: R6.2
Changed lines of the file:
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@@
+	(wire
+		(pts
+			(xy 165.1 102.87) (xy 172.72 102.87)
+		)
+		(stroke
+			(width 0)
+			(type default)
+		)
+	)
 	(wire
 		(pts
@@
 	(wire
 		(pts
-			(xy 187.96 86.36) (xy 187.96 97.79)
-		)
-		(stroke
-			(width 0)
-			(type default)
-		)
-	)
-	(wire
-		(pts
-			(xy 151.13 102.87) (xy 163.83 102.87)
-		)
-		(stroke
-			(width 0)
-			(type default)
-		)
-	)
-	(wire
-		(pts
-			(xy 151.13 105.41) (xy 163.83 105.41)
+			(xy 196.85 86.36) (xy 196.85 97.79)
+		)
+		(stroke
+			(width 0)
+			(type default)
+		)
+	)
+	(wire
+		(pts
+			(xy 151.13 102.87) (xy 157.48 102.87)
+		)
+		(stroke
+			(width 0)
+			(type default)
+		)
+	)
+	(wire
+		(pts
+			(xy 151.13 105.41) (xy 157.48 105.41)
 		)
 		(stroke
@@
 	(wire
 		(pts
-			(xy 151.13 72.39) (xy 162.56 72.39)
-		)
-		(stroke
-			(width 0)
-			(type default)
+			(xy 165.1 105.41) (xy 172.72 105.41)
+		)
+		(stroke
+			(width 0)
+			(type default)
+		)
+	)
+	(wire
+		(pts
+			(xy 151.13 72.39) (xy 171.45 72.39)
+		)
+		(stroke
+			(width 0)
+			(type default)
+		)
+	)
+	(symbol
+		(lib_id "Device:R")
+		(at 161.29 102.87 90)
+		(unit 1)
+		(body_style 1)
+		(exclude_from_sim no)
+		(in_bom yes)
+		(on_board yes)
+		(in_pos_files yes)
+		(dnp no)
+		(fields_autoplaced yes)
+		(property "Reference" "R1"
+			(at 161.29 96.52 90)
+			(show_name no)
+			(do_not_autoplace no)
+			(effects
+				(font
+					(size 1.27 1.27)
+				)
+			)
+		)
+		(property "Value" "27r"
+			(at 161.29 99.06 90)
+			(show_name no)
+			(do_not_autoplace no)
+			(effects
+				(font
+					(size 1.27 1.27)
+				)
+			)
+		)
+		(property "Footprint" "Resistor_SMD:R_0805_2012Metric_Pad1.20x1.40mm_HandSolder"
+			(at 161.29 104.648 90)
+			(hide yes)
+			(show_name no)
+			(do_not_autoplace no)
+			(effects
+				(font
+					(size 1.27 1.27)
+				)
+			)
+		)
+		(property "Datasheet" ""
+			(at 161.29 102.87 0)
+			(hide yes)
+			(show_name no)
+			(do_not_autoplace no)
+			(effects
+				(font
+					(size 1.27 1.27)
+				)
+			)
+		)
+		(property "Description" "Resistor"
+			(at 161.29 102.87 0)
+			(hide yes)
+			(show_name no)
+			(do_not_autoplace no)
+			(effects
+				(font
+					(size 1.27 1.27)
+				)
+			)
+		)
+		(property "LCSC" " C17594 "
+			(at 161.29 102.87 90)
+			(hide yes)
+			(show_name no)
+			(do_not_autoplace no)
+			(effects
+				(font
+					(size 1.27 1.27)
+				)
+			)
+		)
+		(pin "1"
+		)
+		(pin "2"
+		)
+		(instances
+			(project "ESP32_CAN_Board"
+				(path "/25a9066d-fd6c-49ea-904e-882f2dbee539"
+					(reference "R1")
+					(unit 1)
+				)
+			)
+		)
+	)
+	(symbol
+		(lib_id "Device:R")
+		(at 161.29 105.41 90)
+		(unit 1)
+		(body_style 1)
+		(exclude_from_sim no)
+		(in_bom yes)
+		(on_board yes)
+		(in_pos_files yes)
+		(dnp no)
+		(property "Reference" "R6"
+			(at 161.29 108.204 90)
+			(show_name no)
+			(do_not_autoplace no)
+			(effects
+				(font
+					(size 1.27 1.27)
+				)
+			)
+		)
+		(property "Value" "27r"
+			(at 161.29 110.744 90)
+			(show_name no)
+			(do_not_autoplace no)
+			(effects
+				(font
+					(size 1.27 1.27)
+				)
+			)
+		)
+		(property "Footprint" "Resistor_SMD:R_0805_2012Metric_Pad1.20x1.40mm_HandSolder"
+			(at 161.29 107.188 90)
+			(hide yes)
+			(show_name no)
+			(do_not_autoplace no)
+			(effects
+				(font
+					(size 1.27 1.27)
+				)
+			)
+		)
+		(property "Datasheet" ""
+			(at 161.29 105.41 0)
+			(hide yes)
+			(show_name no)
+			(do_not_autoplace no)
+			(effects
+				(font
+					(size 1.27 1.27)
+				)
+			)
+		)
+		(property "Description" "Resistor"
+			(at 161.29 105.41 0)
+			(hide yes)
+			(show_name no)
+			(do_not_autoplace no)
+			(effects
+				(font
+					(size 1.27 1.27)
+				)
+			)
+		)
+		(property "LCSC" " C17594 "
+			(at 161.29 105.41 90)
+			(hide yes)
+			(show_name no)
+			(do_not_autoplace no)
+			(effects
+				(font
+					(size 1.27 1.27)
+				)
+			)
+		)
+		(pin "1"
+		)
+		(pin "2"
+		)
+		(instances
+			(project "ESP32_CAN_Board"
+				(path "/25a9066d-fd6c-49ea-904e-882f2dbee539"
+					(reference "R6")
+					(unit 1)
+				)
+			)
 		)
 	)
@@
 	)
 	(sheet
-		(at 162.56 68.58)
+		(at 171.45 68.58)
 		(size 27.94 17.78)
 		(exclude_from_sim no)
@@
 		)
 		(property "Sheetname" "Power"
-			(at 162.56 67.8684 0)
+			(at 171.45 67.8684 0)
 			(show_name no)
 			(do_not_autoplace no)
@@
 		)
 		(property "Sheetfile" "Power.kicad_sch"
-			(at 162.56 86.9446 0)
+			(at 171.45 86.9446 0)
 			(show_name no)
 			(do_not_autoplace no)
@@
 		)
 		(pin "ESP5vUSB" input
-			(at 187.96 86.36 270)
+			(at 196.85 86.36 270)
 			(effects
 				(font
@@
 		)
 		(pin "ESPPower" input
-			(at 162.56 72.39 180)
+			(at 171.45 72.39 180)
 			(effects
 				(font
@@
 	)
 	(sheet
-		(at 163.83 97.79)
+		(at 172.72 97.79)
 		(size 26.67 21.59)
 		(exclude_from_sim no)
@@
 		)
 		(property "Sheetname" "USBC"
-			(at 163.83 97.0784 0)
+			(at 172.72 97.0784 0)
 			(show_name no)
 			(do_not_autoplace no)
@@
 		)
 		(property "Sheetfile" "USBC.kicad_sch"
-			(at 163.83 119.9646 0)
+			(at 172.72 119.9646 0)
 			(show_name no)
 			(do_not_autoplace no)
@@
 		)
 		(pin "D+" input
-			(at 163.83 102.87 180)
+			(at 172.72 102.87 180)
 			(effects
 				(font
@@
 		)
 		(pin "D-" input
-			(at 163.83 105.41 180)
+			(at 172.72 105.41 180)
 			(effects
 				(font
@@
 		)
 		(pin "ESP5vUSB" input
-			(at 187.96 97.79 90)
-			(effects
-				(font
+			(at 196.85 97.79 90)
+			(effects
+				(font
