File: Schematics/ESP32_CAN_Board/CAN.kicad_sch (KiCad schematic)
At the start: 6 parts, among them U1 SN65HVD230

Commit message: final Draft Completed, In JLPCB Cart
Parts:
- JP1: LCSC C474893 -> (none)
Changed lines of the file:
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@@
 			)
 		)
-		(property "LCSC" "C474893"
+		(property "LCSC" ""
 			(at 140.97 87.63 0)
 			(hide yes)
