File: Schematics/ESP32_CAN_Board/USBC.kicad_sch (KiCad schematic)
At the start: 4 parts, among them J8 USB_C_Receptacle

Commit message: initial design completed
Parts:
- D21: footprint SRV05-4.TCT:SOT95P280X145-6N -> myFootprints:SOT95P280X145-6N
Connections:
- net D-: now also D21.6; no longer D21.3

Commit message: updated ESPBoard
Parts:
- J8: LCSC C49566391 -> C165948
Changed lines of the file:
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@@
 			)
 		)
-		(property "LCSC" "C49566391"
+		(property "LCSC" "C165948"
 			(at 115.57 90.17 0)
 			(hide yes)
